Commit message: The racecar model and corresponding controller configuration have been changed.

File: racecar_sim/racecar_description/urdf/racecar.urdf.xacro (robot description, xacro)
@@ -29,7 +29,7 @@
 <robot name="racecar" xmlns:xacro="http://www.ros.org/wiki/xacro">
   <!-- include sensors -->
-  <xacro:include filename="$(find racecar_description)/urdf/sensors/lidar.xacro" />
+  <!-- <xacro:include filename="$(find racecar_description)/urdf/sensors/lidar.xacro" />
   <xacro:include filename="$(find racecar_description)/urdf/sensors/imu.xacro" />
-  <xacro:include filename="$(find racecar_description)/urdf/sensors/camera.xacro" />
+  <xacro:include filename="$(find racecar_description)/urdf/sensors/camera.xacro" /> -->
   <!-- Degree-to-radian conversions -->
   <xacro:property name="degrees_45" value="0.785398163"/>
@@ -37,8 +37,8 @@
   <!-- chassis_length is measured along the x axis, chassis_width
        along the y axis, and chassis_height along the z axis. -->
-  <xacro:property name="chassis_length" value="0.258"/>
-  <xacro:property name="chassis_width" value="0.168"/>
+  <xacro:property name="chassis_length" value="0.16"/>
+  <xacro:property name="chassis_width" value="0.04"/>
   <xacro:property name="chassis_height" value="0.01"/>
-  <xacro:property name="chassis_mass" value="2.788"/>
+  <xacro:property name="chassis_mass" value="5.788"/>
   <!-- battery_dist is the distance between the inner edges of the
        batteries. battery_comp_depth is the battery compartment depth.
@@ -59,6 +59,6 @@
        axle_length. -->
   <xacro:property name="hub_dia" value="0.09652"/>
-  <xacro:property name="tire_dia" value="0.14605"/>
-  <xacro:property name="tire_width" value="0.0889"/>
+  <xacro:property name="tire_dia" value="0.047"/>
+  <xacro:property name="tire_width" value="0.03"/>
   <xacro:property name="hex_hub_depth" value="0.01445"/>
   <xacro:property name="wheel_mass" value="0.29"/>
@@ -67,9 +67,9 @@
        from a U joint to the corresponding hex hub. wheel_travel is the
        vertical wheel travel. -->
-  <xacro:property name="wheelbase" value="0.335"/>
-  <xacro:property name="hex_hub_dist" value="0.365"/>
+  <xacro:property name="wheelbase" value="0.087"/>
+  <xacro:property name="hex_hub_dist" value="0.125"/>
   <xacro:property name="axle_length" value="0.03"/>
-  <xacro:property name="wheel_travel" value="0.084"/>
-  <xacro:property name="shock_z_offset" value="0.0655"/>
+  <xacro:property name="wheel_travel" value="0.0"/>
+  <xacro:property name="shock_z_offset" value="0.0"/>
   <!-- shock_eff_limit is 2 * ((shock_stroke / 2) * shock_spring_constant) N.
        shock_stroke is 0.028575 meters. shock_spring_constant, an approximation
@@ -90,5 +90,5 @@
        axle_vel_limit = (2 * pi) * (max_speed / (pi * tire_dia)) =
          244.8696 rad/s -->
-  <xacro:property name="axle_eff_limit" value="5.12766"/>
+  <xacro:property name="axle_eff_limit" value="5"/>
   <xacro:property name="axle_vel_limit" value="244.8696"/>
   <!-- These constants are used to simulate a Traxxas 2056 servo operated at
@@ -250,6 +250,5 @@
       <visual>
         <origin xyz="0
-                     ${lr_reflect * (axle_length - (tire_width /
-                     2 - hex_hub_depth))}
+                     0
                      0"/>
         <geometry>
@@ -260,6 +259,5 @@
       <collision>
         <origin xyz="0
-                     ${lr_reflect * (axle_length - (tire_width /
-                     2 - hex_hub_depth))}
+                     0
                      0"/>
         <geometry>
@@ -267,4 +265,9 @@
         </geometry>
       </collision>
+      <gazebo>
+        <mu1>1</mu1> <!-- 静摩擦系数 -->
+        <mu2>0.7</mu2> <!-- 动摩擦系数 -->
+        <min_depth>0.001</min_depth>
+      </gazebo>
       <xacro:thick_walled_tube_inertial
           inner_rad="${hub_dia / 2}" outer_rad="${tire_dia / 2}"
@@ -346,4 +349,10 @@
     </gazebo>
   </xacro:macro>
+  <!-- <link name="world"/>
+  <joint name="fixed_world" type="fixed">
+    <parent link="world"/>
+    <child link="base_footprint"/>
+    <origin xyz="0.0 0.0 0.5"/>
+  </joint> -->
   <link name="base_footprint"/>
   <!-- base_link must have geometry so that its axes can be displayed in
@@ -394,6 +403,6 @@
   </joint>
   <!-- Batteries -->
-  <xacro:battery prefix="left" reflect="1"/>
-  <xacro:battery prefix="right" reflect="-1"/>
+  <!-- <xacro:battery prefix="left" reflect="1"/>
+  <xacro:battery prefix="right" reflect="-1"/> -->
   <!-- Wheels -->
   <xacro:front_wheel lr_prefix="left" fr_prefix="front"
@@ -413,5 +422,5 @@
   </gazebo>
   <!-- layers -->
-  <xacro:layer layer="platform" parent="chassis" m="${layer_mass}" x="${layer_x}" y="${layer_y}" z="${layer_z}">
+  <!-- <xacro:layer layer="platform" parent="chassis" m="${layer_mass}" x="${layer_x}" y="${layer_y}" z="${layer_z}">
     <origin xyz="0 0 ${layer_height}" rpy="0 0 0" />
   </xacro:layer>
@@ -436,4 +445,4 @@
     <child link="camera_link"/>
   </joint>
-  <camera prefix="camera"/>
+  <camera prefix="camera"/> -->
 </robot>

File: racecar_sim/racecar_description/urdf/sensors/imu.xacro (robot description, xacro)
@@ -48,3 +48,4 @@
         </gazebo>
     </xacro:macro>
+    <xacro:imu prefix="imu"/>
 </robot>

File: racecar_sim/racecar_description/urdf/sensors/lidar.xacro (robot description, xacro)
@@ -60,3 +60,4 @@
         </gazebo>
     </xacro:macro>
+    <xacro:lidar prefix="laser"/>
 </robot>

Commit message: Virtual Imu has been added.

File: racecar_sim/racecar_description/urdf/racecar.urdf.xacro (robot description, xacro)
@@ -29,7 +29,7 @@
 <robot name="racecar" xmlns:xacro="http://www.ros.org/wiki/xacro">
   <!-- include sensors -->
-  <!-- <xacro:include filename="$(find racecar_description)/urdf/sensors/lidar.xacro" />
+  <!-- <xacro:include filename="$(find racecar_description)/urdf/sensors/lidar.xacro" /> -->
   <xacro:include filename="$(find racecar_description)/urdf/sensors/imu.xacro" />
-  <xacro:include filename="$(find racecar_description)/urdf/sensors/camera.xacro" /> -->
+  <!-- <xacro:include filename="$(find racecar_description)/urdf/sensors/camera.xacro" /> -->
   <!-- Degree-to-radian conversions -->
   <xacro:property name="degrees_45" value="0.785398163"/>
@@ -424,21 +424,21 @@
   <!-- <xacro:layer layer="platform" parent="chassis" m="${layer_mass}" x="${layer_x}" y="${layer_y}" z="${layer_z}">
     <origin xyz="0 0 ${layer_height}" rpy="0 0 0" />
-  </xacro:layer>
-  <xacro:layer layer="lidar_platform" parent="platform_link" m="${layer_mass}" x="0.12" y="0.10" z="0.01">
+  </xacro:layer> -->
+  <!-- <xacro:layer layer="lidar_platform" parent="platform_link" m="${layer_mass}" x="0.12" y="0.10" z="0.01">
     <origin xyz="0.08 0 ${layer_height}" rpy="0 0 0" />
-  </xacro:layer>
-  <joint name="lidar_joint" type="fixed">
+  </xacro:layer> -->
+  <!-- <joint name="lidar_joint" type="fixed">
     <origin xyz="0 0 0.03" rpy="0 0 0" />
     <parent link="lidar_platform_link"/>
     <child link="laser_link"/>
-  </joint>
-  <lidar prefix="laser"/>
+  </joint> -->
+  <!-- <lidar prefix="laser"/> -->
   <joint name="imu_joint" type="fixed">
-    <origin xyz="0.16 0 0.015" rpy="0 0 0" />
-    <parent link="platform_link"/>
+    <origin xyz="0 0 0" rpy="0 0 0" />
+    <parent link="base_link"/>
     <child link="imu_link"/>
   </joint>
   <imu prefix="imu"/>
-  <joint name="camera_joint" type="fixed">
+  <!-- <joint name="camera_joint" type="fixed">
     <origin xyz="0.16 0 0.05" rpy="0 0 0" />
     <parent link="platform_link"/>

File: racecar_sim/racecar_description/urdf/sensors/imu.xacro (robot description, xacro)
@@ -26,5 +26,5 @@
         </link>
         <gazebo reference="${prefix}_link">
-            <material>Gazebo/Black</material>
+            <material>Gazebo/Blue</material>
         </gazebo>
         <gazebo reference="${prefix}_link">

Commit message: Rear driving mode has been added.

File: racecar_sim/racecar_description/urdf/racecar.urdf.xacro (robot description, xacro)
@@ -349,10 +349,10 @@
     </gazebo>
   </xacro:macro>
-  <!-- <link name="world"/>
+  <link name="world"/>
   <joint name="fixed_world" type="fixed">
     <parent link="world"/>
     <child link="base_footprint"/>
     <origin xyz="0.0 0.0 0.5"/>
-  </joint> -->
+  </joint>
   <link name="base_footprint"/>
   <!-- base_link must have geometry so that its axes can be displayed in

Commit message: Odometry calculator based on wheel encoders has been implemented. An EKF filter node has been implemented to fuse imu datas and odometry datas.

File: racecar_sim/racecar_description/urdf/racecar.urdf.xacro (robot description, xacro)
@@ -40,5 +40,5 @@
   <xacro:property name="chassis_width" value="0.04"/>
   <xacro:property name="chassis_height" value="0.01"/>
-  <xacro:property name="chassis_mass" value="5.788"/>
+  <xacro:property name="chassis_mass" value="10.788"/>
   <!-- battery_dist is the distance between the inner edges of the
        batteries. battery_comp_depth is the battery compartment depth.
@@ -58,8 +58,8 @@
        is a "zero offset" wheel. hex_hub_depth = tire_width / 2 -
        axle_length. -->
-  <xacro:property name="hub_dia" value="0.09652"/>
+  <xacro:property name="hub_dia" value="0.0"/>
   <xacro:property name="tire_dia" value="0.047"/>
   <xacro:property name="tire_width" value="0.03"/>
-  <xacro:property name="hex_hub_depth" value="0.01445"/>
+  <xacro:property name="hex_hub_depth" value="0.0"/>
   <xacro:property name="wheel_mass" value="0.29"/>
   <!-- hex_hub_dist is the distance between left and right hex hubs when
@@ -67,7 +67,7 @@
        from a U joint to the corresponding hex hub. wheel_travel is the
        vertical wheel travel. -->
-  <xacro:property name="wheelbase" value="0.087"/>
+  <xacro:property name="wheelbase" value="0.174"/>
   <xacro:property name="hex_hub_dist" value="0.125"/>
-  <xacro:property name="axle_length" value="0.03"/>
+  <xacro:property name="axle_length" value="0.00"/>
   <xacro:property name="wheel_travel" value="0.0"/>
   <xacro:property name="shock_z_offset" value="0.0"/>
@@ -198,5 +198,5 @@
   <xacro:macro name="shock"
                params="lr_prefix fr_prefix lr_reflect fr_reflect child">
-    <joint name="${lr_prefix}_${fr_prefix}_shock" type="prismatic">
+    <joint name="${lr_prefix}_${fr_prefix}_shock" type="fixed">
       <parent link="chassis"/>
       <child link="${child}"/>
@@ -208,5 +208,5 @@
              effort="${shock_eff_limit}" velocity="${shock_vel_limit}"/>
     </joint>
-    <transmission name="${lr_prefix}_${fr_prefix}_shock_trans">
+    <!-- <transmission name="${lr_prefix}_${fr_prefix}_shock_trans">
       <type>transmission_interface/SimpleTransmission</type>
       <joint name="${lr_prefix}_${fr_prefix}_shock">
@@ -214,10 +214,8 @@
       </joint>
       <actuator name="${lr_prefix}_${fr_prefix}_shock_act">
-        <!-- This hardwareInterface element exists for compatibility
-             with ROS Hydro. -->
         <hardwareInterface>hardware_interface/EffortJointInterface</hardwareInterface>
         <mechanicalReduction>1</mechanicalReduction>
       </actuator>
-    </transmission>
+    </transmission> -->
   </xacro:macro>
   <!-- The "wheel" macro defines an axle carrier, axle, and wheel. -->
@@ -267,5 +265,5 @@
       <gazebo>
         <mu1>1</mu1> <!-- 静摩擦系数 -->
-        <mu2>0.7</mu2> <!-- 动摩擦系数 -->
+        <mu2>1</mu2> <!-- 动摩擦系数 -->
         <min_depth>0.001</min_depth>
       </gazebo>
@@ -349,10 +347,10 @@
     </gazebo>
   </xacro:macro>
-  <link name="world"/>
+  <!-- <link name="world"/>
   <joint name="fixed_world" type="fixed">
     <parent link="world"/>
     <child link="base_footprint"/>
     <origin xyz="0.0 0.0 0.5"/>
-  </joint>
+  </joint> -->
   <link name="base_footprint"/>
   <!-- base_link must have geometry so that its axes can be displayed in

Commit message: Create the ros bag data processor node.

File: racecar_sim/racecar_description/urdf/racecar.urdf.xacro (robot description, xacro)
@@ -433,5 +433,5 @@
   <!-- <lidar prefix="laser"/> -->
   <joint name="imu_joint" type="fixed">
-    <origin xyz="0 0 0" rpy="0 0 0" />
+    <origin xyz="0 0 0" rpy="3.1415926 0 0" />
     <parent link="base_link"/>
     <child link="imu_link"/>
